Commit message: Add files via upload

File: xacro/go2_generated2.urdf (robot description, URDF)
Before this commit: robot go2, 23 links, 22 joints
Links:
- removed link camera
- removed link camera_link_optical
- removed link velodyne
- removed link velodyne_base_link
- added link hokuyo_frame, mass 0.270; collision box size=0.058 0.058 0.087; visual mesh filename=package://hector_sensors_description/meshes/hokuyo_utm30lx/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
- link imu_link: geometry collision box size=.001 .001 .001; visual box size=0.001 0.001 0.001
Joints:
- removed joint camera_joint
- removed joint camera_optical_joint
- removed joint velodyne_base_mount_joint
- removed joint velodyne_base_scan_joint
- added joint hokuyo_joint: type fixed, parent trunk, child hokuyo_frame, origin xyz=0.0 0.0 0.096 rpy=0 0 0

File: xacro/go2_velodyne_description (copy).urdf (robot description, URDF)
Before this commit: robot go2, 23 links, 22 joints
Links:
- removed link camera
- removed link camera_link_optical
- link imu_link: geometry collision box size=.001 .001 .001; visual box size=0.001 0.001 0.001
Joints:
- removed joint camera_joint
- removed joint camera_optical_joint
